File: adapter/everstar.kicad_pcb (KiCad board)
At the start: 2 copper layers, 90.2 x 62.2 mm, 9 parts, among them J1 EV29LV640, J2 EV29LV160, J3 M27V322, J4 A21

Commit message: Order number position on bottom layer for JLCPCB
Other:
- board text added: "JLCJLCJLCJLC"
Changed lines of the file:
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@@
   (gr_arc (start 55.88 121.285) (mid 51.838885 119.611115) (end 50.165 115.57)
     (stroke (width 0.1) (type default)) (layer "Edge.Cuts"))
+  (gr_text "JLCJLCJLCJLC" (at 133.35 119.38 -90) (layer "B.SilkS")
+    (effects (font (size 1 1) (thickness 0.15)) (justify left bottom mirror))
+  )
   (gr_text "Everstar / IGS\nROM adapter\n\nbuffi - 2024" (at 51.435 109.855) (layer "F.SilkS")
     (effects (font (size 1.3 1.3) (thickness 0.25) bold) (justify left))
